File: foc_board/foc_board.kicad_sch (KiCad schematic)
At the start: 9 parts, among them U1 STM32G431CBUx, U2 STM32G431CBUx, U3 TCAN3413DDFR, Y1 16MHz

Commit message: 10/25 journal update
Parts:
- removed C1, C2: 12pF, Capacitor_SMD:C_0603_1608Metric, symbol Device:C_Small
- removed C3: 100nF, symbol Device:C_Small
- removed R1, R2: 120, symbol Device:R
- removed U1, U2: STM32G431CBUx, Package_DFN_QFN:QFN-48-1EP_7x7mm_P0.5mm_EP5.6x5.6mm, symbol MCU_ST_STM32G4:STM32G431CBUx
- removed U3: TCAN3413DDFR, SOT-23-THIN-8_DDF_TEX, symbol TCAN3413:PTCAN3413DDFR
- removed Y1: 16MHz, Capacitor_SMD:C_0402_1005Metric, symbol Device:Crystal_GND24
Other:
- added sheet CAN (can.kicad_sch)
- added sheet MCU (mcu.kicad_sch)
